File: V0_Display/KiCad/V0_Display.sch (KiCad schematic (older format))
At the start: 28 parts, among them J1 USB_B_Micro, J2 I2C Header 1, J3 Conn_01x03, J4 Conn_01x02, J5 SWD Header, J7 USB_Header, J8 Conn_01x02, SW5 SW_SPST, SW6 SW_SPST, SW7 Rotary_Encoder_Switch, U1 AP2127K-3.3, U2 STM32F042F6Px, U3 74LVC1G17

Commit message: Microcontroller change
Changed the STM32F042 microcontroller for an ATmega32U4, given the scarcity of the former due to the pandemic of Covid-19.
Parts:
- removed C1, C2: 4.7uF, V0-Display:C_0805_2012Metric, symbol Device:C
- removed C4: 0.1uF, V0-Display:C_0805_2012Metric, symbol V0_Display:C
- removed GPIO1, J3: Conn_01x03, V0-Display:PinHeader_1x03_P2.54mm_Vertical, symbol V0_Display:Conn_01x03
- removed J4: Conn_01x02, V0-Display:PinHeader_1x02_P2.54mm_Vertical, symbol V0_Display:Conn_01x02
- removed J5: SWD Header, V0-Display:PinHeader_2x05_P1.27mm_Vertical_SMD, symbol V0_Display:Conn_02x05_Odd_Even
- removed U1: AP2127K-3.3, V0-Display:SOT-23-5, symbol V0_Display:AP2127K-3.3
- removed U2: STM32F042F6Px, V0-Display:TSSOP-20_4.4x6.5mm_P0.65mm, symbol V0_Display:STM32F042F6Px
- removed U3: 74LVC1G17, V0-Display:SOT-753, symbol V0_Display:74LVC1G17
- added C1, C2, C7, C8: 0.1µF, V0-Display:C_0805_2012Metric, symbol V0_Display:C
- added C4, C5: 8pF, V0-Display:C_0805_2012Metric, symbol Device:C
- added C6: 1µF, V0-Display:C_0805_2012Metric, symbol V0_Display:C
- added J3: Conn_01x11, Pin_Headers:Pin_Header_Straight_1x11_Pitch2.54mm, symbol Connector_Generic:Conn_01x11
- added J6: ICSP, Pin_Headers:Pin_Header_Straight_2x03_Pitch2.54mm, symbol Connector_Generic:Conn_02x03_Odd_Even
- added J7: JTAG, Pin_Headers:Pin_Header_Straight_2x05_Pitch1.27mm, symbol Connector_Generic:Conn_02x05_Odd_Even
- added R4: 10K, V0-Display:R_0805_2012Metric, symbol V0_Display:R
- added U1: ATmega32U4-AU, Housings_QFP:TQFP-44_10x10mm_Pitch0.8mm, symbol MCU_Microchip_ATmega:ATmega32U4-AU
- added Y1: 16MHz, Crystals:Crystal_HC50_Vertical, symbol Device:Crystal
- C3: value 0.1uF -> 0.1µF
- R2, R3: value 10K -> 22R
- renumbered J7 to J2, J2 to J4, J8 to J5, SW5 to SW1, SW7 to SW2, SW6 to SW3
Connections:
- net labels added: GPIO10, GPIO11, GPIO5, GPIO6, GPIO7, GPIO8, GPIO9, MISO, MOSI, SCLK, TCK, TDI, TDO, TMS
- net labels removed: +3V3, BOOT0, SWDCLK, SWDIO
- wire segments 86 -> 109
- no-connect marks 4 -> 3
